File: nitinolDriver.sch (EAGLE design)
At the start: 25 parts

Commit message: changed to 16A NMOSFETs
Parts:
- removed R6, R7: 0, fab:RES-US1206FAB
- removed T1, T2: (no value), fab:NMOSFETSOT23
- added T3, T4: (no value), fab:NMOSFETTO252
- R1, R2: value 150 -> 100
Connections:
- removed net N$5: PAD4.P, R7.2
- removed net N$8: PAD2.P, R6.2
- net GND: now also T3.S, T4.S; no longer T1.S, T2.S
- net N$1: now also R2.2, T4.G; no longer R1.2, T1.G
- net N$11: now also PAD4.P, T4.D; no longer R7.1, T2.D
- net N$14: now also PAD2.P, T3.D; no longer R6.1, T1.D
- net N$2: now also R1.2, T3.G; no longer R2.2, T2.G
Changed lines of the file:
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@@
 <parts>
 <part name="U$1" library="fab" deviceset="ATTINY45" device="SI"/>
-<part name="R1" library="fab" deviceset="RES-US" device="1206FAB" value="150"/>
-<part name="R2" library="fab" deviceset="RES-US" device="1206FAB" value="150"/>
+<part name="R1" library="fab" deviceset="RES-US" device="1206FAB" value="100"/>
+<part name="R2" library="fab" deviceset="RES-US" device="1206FAB" value="100"/>
 <part name="R3" library="fab" deviceset="RES-US" device="1206FAB" value="10k"/>
 <part name="R4" library="fab" deviceset="RES-US" device="1206FAB" value="10k"/>
 <part name="R5" library="fab" deviceset="RES-US" device="1206FAB" value="10k"/>
-<part name="R6" library="fab" deviceset="RES-US" device="1206FAB" value="0"/>
-<part name="R7" library="fab" deviceset="RES-US" device="1206FAB" value="0"/>
-<part name="T1" library="fab" deviceset="NMOSFET" device="SOT23"/>
-<part name="T2" library="fab" deviceset="NMOSFET" device="SOT23"/>
 <part name="R8" library="fab" deviceset="RES-US" device="1206FAB" value="100"/>
 <part name="R9" library="fab" deviceset="RES-US" device="1206FAB" value="100"/>
@@
 <part name="GND11" library="supply1" deviceset="GND" device=""/>
 <part name="P+7" library="supply1" deviceset="V+" device=""/>
+<part name="T3" library="fab" deviceset="NMOSFET" device="TO252"/>
+<part name="T4" library="fab" deviceset="NMOSFET" device="TO252"/>
 </parts>
 <sheets>
@@
 <instance part="R4" gate="G$1" x="190.5" y="48.26" rot="R90"/>
 <instance part="R5" gate="G$1" x="-2.54" y="63.5" rot="R90"/>
-<instance part="R6" gate="G$1" x="160.02" y="86.36" rot="R90"/>
-<instance part="R7" gate="G$1" x="210.82" y="86.36" rot="R90"/>
-<instance part="T1" gate="A" x="160.02" y="71.12"/>
-<instance part="T2" gate="A" x="210.82" y="71.12"/>
 <instance part="R8" gate="G$1" x="132.08" y="58.42" rot="R90"/>
 <instance part="R9" gate="G$1" x="177.8" y="58.42" rot="R90"/>
@@
 <instance part="GND11" gate="1" x="114.3" y="86.36"/>
 <instance part="P+7" gate="1" x="101.6" y="99.06"/>
+<instance part="T3" gate="A" x="160.02" y="71.12"/>
+<instance part="T4" gate="A" x="210.82" y="71.12"/>
 </instances>
 <busses>
 </busses>
 <nets>
-<net name="N$1" class="0">
-<segment>
-<pinref part="R1" gate="G$1" pin="2"/>
-<pinref part="T1" gate="A" pin="G"/>
-</segment>
-</net>
-<net name="N$2" class="0">
-<segment>
-<pinref part="R2" gate="G$1" pin="2"/>
-<pinref part="T2" gate="A" pin="G"/>
-</segment>
-</net>
 <net name="N$3" class="0">
 <segment>
@@
 <net name="N$11" class="0">
 <segment>
-<pinref part="T2" gate="A" pin="D"/>
-<pinref part="R7" gate="G$1" pin="1"/>
-<wire x1="210.82" y1="76.2" x2="210.82" y2="81.28" width="0.1524" layer="91"/>
+<pinref part="T4" gate="A" pin="D"/>
+<pinref part="PAD4" gate="1" pin="P"/>
+<wire x1="210.82" y1="76.2" x2="210.82" y2="96.52" width="0.1524" layer="91"/>
 </segment>
 </net>
 <net name="N$14" class="0">
 <segment>
-<pinref part="R6" gate="G$1" pin="1"/>
-<pinref part="T1" gate="A" pin="D"/>
-<wire x1="160.02" y1="81.28" x2="160.02" y2="76.2" width="0.1524" layer="91"/>
+<pinref part="T3" gate="A" pin="D"/>
+<pinref part="PAD2" gate="1" pin="P"/>
+<wire x1="160.02" y1="76.2" x2="160.02" y2="96.52" width="0.1524" layer="91"/>
 </segment>
 </net>
@@
 </segment>
 <segment>
-<pinref part="T1" gate="A" pin="S"/>
 <wire x1="160.02" y1="66.04" x2="160.02" y2="27.94" width="0.1524" layer="91"/>
 <pinref part="GND3" gate="1" pin="GND"/>
+<pinref part="T3" gate="A" pin="S"/>
 </segment>
 <segment>
@@
 </segment>
 <segment>
-<pinref part="T2" gate="A" pin="S"/>
 <wire x1="210.82" y1="66.04" x2="210.82" y2="27.94" width="0.1524" layer="91"/>
 <pinref part="GND6" gate="1" pin="GND"/>
+<pinref part="T4" gate="A" pin="S"/>
 </segment>
 <segment>
@@
 </segment>
 </net>
-<net name="N$5" class="0">
-<segment>
-<pinref part="R7" gate="G$1" pin="2"/>
-<pinref part="PAD4" gate="1" pin="P"/>
-<wire x1="210.82" y1="91.44" x2="210.82" y2="96.52" width="0.1524" layer="91"/>
-</segment>
-</net>
-<net name="N$8" class="0">
-<segment>
-<pinref part="R6" gate="G$1" pin="2"/>
-<pinref part="PAD2" gate="1" pin="P"/>
-<wire x1="160.02" y1="91.44" x2="160.02" y2="96.52" width="0.1524" layer="91"/>
-</segment>
-</net>
+<net name="N$1" class="0">
+<segment>
+<pinref part="R2" gate="G$1" pin="2"/>
+<pinref part="T4" gate="A" pin="G"/>
+</segment>
+</net>
+<net name="N$2" class="0">
+<segment>
+<pinref part="R1" gate="G$1" pin="2"/>
+<pinref part="T3" gate="A" pin="G"/>
+</segment>
+</net>
